File: capteur_ultra-sonic/docs/ultra-sonic/ultra-sonic.kicad_sch (KiCad schematic)
At the start: 6 parts, among them J1 Capteur Ultrasonic, U1 ESP32-DevKitC, U2 ER_OLEDM0.91_1x-I2C

Commit message: Météo
Connections:
- net at BZ1.2 (-), J1.GND (Pin_4), R2.2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: now also U2.1 (GND)
Changed lines of the file:
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@@
+	)
+	(junction
+		(at 177.8 124.46)
+		(diameter 0)
+		(color 0 0 0 0)
 	)
 	(junction
@@
 	(wire
 		(pts
+			(xy 196.85 88.9) (xy 196.85 124.46)
+		)
+		(stroke
+			(width 0)
+			(type default)
+		)
+	)
+	(wire
+		(pts
 			(xy 182.88 76.2) (xy 182.88 83.82)
 		)
@@
 		)
 		(stroke
+			(width 0)
+			(type default)
+		)
+	)
+	(wire
+		(pts
+			(xy 196.85 124.46) (xy 177.8 124.46)
+		)
+		(stroke
