File: carte_rfid/docs/carte_rfid/carte_rfid.kicad_sch (KiCad schematic)
At the start: 4 parts, among them U1 ESP32-DevKit, U2 OLED

Commit message: Ajout 2 leds (Accès autorisé/réfusé)
Parts:
- added LED: VERT, symbol Device:LED
- added LED: ROUGE, symbol Device:LED
- added R1, R2: 220, Package_DIP:DIP-8_W7.62mm, symbol Device:R
Connections:
- net at BZ1.2 (-), RC522.6 (GND), U1.14 (GND)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: now also LED.1 (K), LED.1 (K)
- net at U1.12 (MTMS/GPIO14/ADC2_CH6): now also R2.1
- net at U1.13 (MTDI/GPIO12/ADC2_CH5): now also R1.1
- new net: LED.2 (A), R2.2
- new net: LED.2 (A), R1.2
Other:
- moved on the sheet: BZ1, RC522, U1, U2
